File: keyboard_keyboard/kicad/keyboard_keyboard.kicad_sch (KiCad schematic)
At the start: 331 parts, among them J1 TYPE-C-31-M-12, J2 JST_SH, SW1 TS-1187A-B-A-B, SW2 TS-1187A-B-A-B, U1 USBLC6-2SC6, U2 TLV75733PDBV, U3 XC6206P332MR-G, U4 AT32F405RCT7, Y1 X322512MSB4SI

Commit message: wip pcb
Parts:
- added A1: Electrosmith_Daisy_Seed_Rev4, Module:Electrosmith_Daisy_Seed, symbol MCU_Module:Electrosmith_Daisy_Seed_Rev4
- added AM10, AM11: SN74LV4051A, Package_SO:TSSOP-16_4.4x5mm_P0.65mm, symbol 4xxx:4051
- added C161, C162: 100n, Capacitor_SMD:C_0402_1005Metric, symbol Device:C
Connections:
- net +3.3VA: now also AM10.16 (VDD), AM11.16 (VDD), C161.1, C162.1
- net GND: now also AM10.6 (Inh), AM10.7 (VEE), AM10.8 (VSS), AM11.6 (Inh), AM11.7 (VEE), AM11.8 (VSS), C161.2, C162.2
- net MUX_OUT_1: now also A1.22 (ADC_0)
- net MUX_OUT_2: now also A1.23 (ADC_1)
- net MUX_OUT_3: now also A1.24 (ADC_2)
- net MUX_OUT_4: now also A1.25 (ADC_3)
- net MUX_OUT_5: now also A1.26 (ADC_4)
- net MUX_OUT_6: now also A1.27 (ADC_5)
- net MUX_OUT_7: now also A1.28 (ADC_6)
- net MUX_OUT_8: now also A1.29 (DAC_OUT2)
- net MUX_OUT_9: now also A1.30 (DAC_OUT1)
- net MUX_SELECT_0: now also AM10.11 (A), AM11.11 (A)
- net MUX_SELECT_1: now also AM10.10 (B), AM11.10 (B)
- net MUX_SELECT_2: now also AM10.9 (C), AM11.9 (C)
- new net MUX_OUT_10: A1.31 (SAI2_MCLK), AM10.3 (X)
- new net MUX_OUT_11: A1.32 (SAI2_SD_B), AM11.3 (X)
