File: keyboard_keyboard/kicad/keyboard_keyboard.kicad_sch (KiCad schematic)
At the start: 336 parts, among them J1 TYPE-C-31-M-12, J2 JST_SH, SW1 TS-1187A-B-A-B, SW2 TS-1187A-B-A-B, U1 USBLC6-2SC6, U2 TLV75733PDBV, U3 XC6206P332MR-G, U4 AT32F405RCT7, Y1 X322512MSB4SI

Commit message: more routing
Parts:
- added C163, C165: 100n, Capacitor_SMD:C_0402_1005Metric, symbol Device:C
- added C164, C166: 4.7n, Capacitor_SMD:C_0402_1005Metric, symbol Device:C
- added HE70, HE71: MT9102ET, Package_TO_SOT_SMD:SOT-23-3, symbol HE60:MT9102ET
Connections:
- net +3.3VA: now also C163.1, C165.1, HE70.1 (VCC), HE71.1 (VCC)
- net GND: now also C163.2, C164.2, C165.2, C166.2, HE70.3 (GND), HE71.3 (GND)
- net HE69: now also C164.1, C166.1, HE70.2 (OUT), HE71.2 (OUT)
Other:
- moved on the sheet: A1, AM1, AM10, AM11, AM2, AM3, AM4, AM5, AM6, AM7, AM8, AM9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

Commit message: more keys
Parts:
- added C167, C169, C171, C173, C175, C177, C179, C181, C183, C185, C187, C189, C191, C193, C195, C197, C199, C201, C203, C205, C207, C209, C211, C213, C215, C217, C219, C221, C223: 100n, Capacitor_SMD:C_0402_1005Metric, symbol Device:C
- added C168, C170, C172, C174, C176, C178, C180, C182, C184, C186, C188, C190, C192, C194, C196, C198, C200, C202, C204, C206, C208, C210, C212, C214, C216, C218, C220, C222, C224: 4.7n, Capacitor_SMD:C_0402_1005Metric, symbol Device:C
- added HE100, HE72, HE73, HE74, HE75, HE76, HE77, HE78, HE79, HE80, HE81, HE82, HE83, HE84, HE85, HE86, HE87, HE88, HE89, HE90, HE91, HE92, HE93, HE94, HE95, HE96, HE97, HE98, HE99: MT9102ET, Package_TO_SOT_SMD:SOT-23-3, symbol HE60:MT9102ET
- MX14: value 1U -> 1.5U; footprint HE60:MX-1U -> HE60:MX-1.5U
- MX15: value 2U -> 1U; footprint HE60:MX-2U -> HE60:MX-1U
- MX17, MX63, MX71, MX75: value 1.5U -> 1U; footprint HE60:MX-1.5U -> HE60:MX-1U
- MX31: value 1.75U -> 1U; footprint HE60:MX-1.75U -> HE60:MX-1U
- MX43: value 2.25U -> 1.5U; footprint HE60:MX-2.25U -> HE60:MX-1.5U
- MX44: value 2.25U -> 1u; footprint HE60:MX-2.25U -> HE60:MX-1U
- MX55: value 1.75U -> 15U; footprint HE60:MX-1.75U -> HE60:MX-1U
- MX56: value 2.75U -> 1U; footprint HE60:MX-2.75U -> HE60:MX-1U
- MX58, MX60, MX62, MX72, MX74, MX76: value 1.25U -> 1U; footprint HE60:MX-1.25U -> HE60:MX-1U
- MX65: value 2.25U -> 1U; footprint HE60:MX-2.25U-ReversedStabilizers -> HE60:MX-1U
- MX66: value 6.25U -> 1U; footprint HE60:MX-6.25U-ReversedStabilizers -> HE60:MX-1U
- MX67: value 7U -> 1U; footprint HE60:MX-7U-ReversedStabilizers -> HE60:MX-1U
- MX68: value 2.75U -> 1U; footprint HE60:MX-2.75U-ReversedStabilizers -> HE60:MX-1U
- MX70: value 1.25U -> 1.5U; footprint HE60:MX-1.25U -> HE60:MX-1.5U
Connections:
- net +3.3VA: now also C167.1, C169.1, C171.1, C173.1, C175.1, C177.1, C179.1, C181.1, C183.1, C185.1, C187.1, C189.1, C191.1, C193.1, C195.1, C197.1, C199.1, C201.1, C203.1, C205.1, C207.1, C209.1, C211.1, C213.1, C215.1, C217.1, C219.1, C221.1, C223.1, HE100.1 (VCC), HE72.1 (VCC), HE73.1 (VCC), HE74.1 (VCC), HE75.1 (VCC), HE76.1 (VCC), HE77.1 (VCC), HE78.1 (VCC), HE79.1 (VCC), HE80.1 (VCC), HE81.1 (VCC), HE82.1 (VCC), HE83.1 (VCC), HE84.1 (VCC), HE85.1 (VCC), HE86.1 (VCC), HE87.1 (VCC), HE88.1 (VCC), HE89.1 (VCC), HE90.1 (VCC), HE91.1 (VCC), HE92.1 (VCC), HE93.1 (VCC), HE94.1 (VCC), HE95.1 (VCC), HE96.1 (VCC), HE97.1 (VCC), HE98.1 (VCC), HE99.1 (VCC)
- net GND: now also C167.2, C168.2, C169.2, C170.2, C171.2, C172.2, C173.2, C174.2, C175.2, C176.2, C177.2, C178.2, C179.2, C180.2, C181.2, C182.2, C183.2, C184.2, C185.2, C186.2, C187.2, C188.2, C189.2, C190.2, C191.2, C192.2, C193.2, C194.2, C195.2, C196.2, C197.2, C198.2, C199.2, C200.2, C201.2, C202.2, C203.2, C204.2, C205.2, C206.2, C207.2, C208.2, C209.2, C210.2, C211.2, C212.2, C213.2, C214.2, C215.2, C216.2, C217.2, C218.2, C219.2, C220.2, C221.2, C222.2, C223.2, C224.2, HE100.3 (GND), HE72.3 (GND), HE73.3 (GND), HE74.3 (GND), HE75.3 (GND), HE76.3 (GND), HE77.3 (GND), HE78.3 (GND), HE79.3 (GND), HE80.3 (GND), HE81.3 (GND), HE82.3 (GND), HE83.3 (GND), HE84.3 (GND), HE85.3 (GND), HE86.3 (GND), HE87.3 (GND), HE88.3 (GND), HE89.3 (GND), HE90.3 (GND), HE91.3 (GND), HE92.3 (GND), HE93.3 (GND), HE94.3 (GND), HE95.3 (GND), HE96.3 (GND), HE97.3 (GND), HE98.3 (GND), HE99.3 (GND)
- net HE69: no longer C164.1, C166.1, HE70.2 (OUT), HE71.2 (OUT)
- net HE74: now reaches AM10.1 (X4)
- net HE74: now also C172.1, HE74.2 (OUT)
- net HE70: now reaches AM10.12 (X3)
- net HE70: now also C164.1, HE70.2 (OUT)
- net HE73: now reaches AM10.13 (X0)
- net HE73: now also C170.1, HE73.2 (OUT)
- net HE72: now reaches AM10.14 (X1)
- net HE72: now also C168.1, HE72.2 (OUT)
- net HE71: now reaches AM10.15 (X2)
- net HE71: now also C166.1, HE71.2 (OUT)
- net HE75: now reaches AM10.2 (X6)
- net HE75: now also C174.1, HE75.2 (OUT)
- net HE76: now reaches AM10.4 (X7)
- net HE76: now also C176.1, HE76.2 (OUT)
- net HE77: now reaches AM10.5 (X5)
- net HE77: now also C178.1, HE77.2 (OUT)
- new net HE100: C224.1, HE100.2 (OUT)
- new net HE78: C180.1, HE78.2 (OUT)
- new net HE79: C182.1, HE79.2 (OUT)
- new net HE80: C184.1, HE80.2 (OUT)
- new net HE81: C186.1, HE81.2 (OUT)
- new net HE82: C188.1, HE82.2 (OUT)
- new net HE83: C190.1, HE83.2 (OUT)
- new net HE84: C192.1, HE84.2 (OUT)
- new net HE85: C194.1, HE85.2 (OUT)
- new net HE86: C196.1, C198.1, HE86.2 (OUT), HE87.2 (OUT)
- new net HE88: C200.1, HE88.2 (OUT)
- new net HE89: C202.1, HE89.2 (OUT)
- new net HE90: C204.1, HE90.2 (OUT)
- new net HE91: C206.1, HE91.2 (OUT)
- new net HE92: C208.1, HE92.2 (OUT)
- new net HE93: C210.1, HE93.2 (OUT)
- new net HE94: C212.1, HE94.2 (OUT)
- new net HE95: C214.1, HE95.2 (OUT)
- new net HE96: C216.1, HE96.2 (OUT)
- new net HE97: C218.1, HE97.2 (OUT)
- new net HE98: C220.1, HE98.2 (OUT)
- new net HE99: C222.1, HE99.2 (OUT)
Other:
- moved on the sheet: C1, C10, C100, C101, C102, C103, C104, C105, C106, C107, C108, C109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

Commit message: more keys
Parts:
- added MX100, MX77, MX78, MX79, MX80, MX81, MX82, MX83, MX84, MX85, MX86, MX87, MX88, MX89, MX90, MX91, MX92, MX93, MX94, MX95, MX96, MX97, MX98, MX99: 1U, HE60:MX-1U, symbol Mechanical:MountingHole
Other:
- moved on the sheet: C185, C186, C187, C188, C189, C190, C191, C192, C193, C194, C195, C196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

Commit message: feat: place everything*
Parts:
- removed C150, C151: 2.2u, Capacitor_SMD:C_0603_1608Metric, symbol Device:C
- removed C152, C153: 30p, Capacitor_SMD:C_0603_1608Metric, symbol Device:C
- removed C154, C155, C156, C158, C160: 100n, Capacitor_SMD:C_0402_1005Metric, symbol Device:C
- removed C157: 10u, Capacitor_SMD:C_0603_1608Metric, symbol Device:C
- removed C159: 1u, Capacitor_SMD:C_0603_1608Metric, symbol Device:C
- removed F1: BSMD0805-050-24V, Fuse:Fuse_0805_2012Metric, symbol Device:Polyfuse
- removed J1: TYPE-C-31-M-12, Connector_USB:USB_C_Receptacle_HRO_TYPE-C-31-M-12, symbol Connector:USB_C_Receptacle_USB2.0_16P
- removed J2: JST_SH, Connector_JST:JST_SH_SM04B-SRSS-TB_1x04-1MP_P1.00mm_Horizontal, symbol Connector_Generic_MountingPin:Conn_01x04_MountingPin
- removed PCB1: H60, HE60:H60, symbol Mechanical:MountingHole_Pad
- removed R1, R2: 5.1k, Resistor_SMD:R_0402_1005Metric, symbol Device:R
- removed R3, R4: 12k, Resistor_SMD:R_0402_1005Metric, symbol Device:R
- removed SW1, SW2: TS-1187A-B-A-B, Button_Switch_SMD:SW_Push_1P1T_XKB_TS-1187A, symbol Switch:SW_Push
- removed TH1, TH2: ToolingHole, HE60:ToolingHole, symbol Mechanical:MountingHole
- removed U1: USBLC6-2SC6, Package_TO_SOT_SMD:SOT-23-6, symbol Power_Protection:USBLC6-2SC6
- removed U2: TLV75733PDBV, Package_TO_SOT_SMD:SOT-23-5, symbol Regulator_Linear:TLV75733PDBV
- removed U3: XC6206P332MR-G, Package_TO_SOT_SMD:SOT-23-3, symbol Regulator_Linear:XC6206PxxxMR
- removed U4: AT32F405RCT7, Package_QFP:LQFP-64_10x10mm_P0.5mm, symbol HE60:AT32F405RxT7
- removed Y1: X322512MSB4SI, Crystal:Crystal_SMD_3225-4Pin_3.2x2.5mm, symbol Device:Crystal_GND24
- added AM12, AM13: SN74LV4051A, Package_SO:TSSOP-16_4.4x5mm_P0.65mm, symbol 4xxx:4051
- added D1, D2, D3: LED, LED_THT:LED_D3.0mm, symbol Device:LED
- added J1, J2: AudioJack3_Ground, Connector_Audio:Jack_3.5mm_PJ320E_Horizontal, symbol Connector_Audio:AudioJack3_Ground
- added R1, R2, R3: R_Small_US, Resistor_THT:R_Axial_DIN0204_L3.6mm_D1.6mm_P7.62mm_Horizontal, symbol Device:R_Small_US
- added RV1, RV10, RV11, RV12, RV2, RV3, RV4, RV5, RV6, RV7, RV8, RV9: R_Potentiometer_Trim_US, Potentiometer_THT:Potentiometer_Alpha_RD901F-40-00D_Single_Vertical, symbol Device:R_Potentiometer_Trim_US
- added SW3, SW4, SW5: RotaryEncoder_Switch, Rotary_Encoder:RotaryEncoder_Alps_EC11E_Vertical_H20mm, symbol Device:RotaryEncoder_Switch
- C148, C149: value 2.2u -> 100n; footprint Capacitor_SMD:C_0603_1608Metric -> Capacitor_SMD:C_0402_1005Metric
- MX55: value 15U -> 1U
Connections:
- net +5V is gone; now on net +3.3VA: C148.1
- net +3.3VA: now also AM12.16 (VDD), AM13.16 (VDD), RV1.1, RV10.1, RV11.1, RV12.1, RV2.1, RV3.1, RV4.1, RV5.1, RV6.1, RV7.1, RV8.1, RV9.1
- net GND: now also AM12.6 (Inh), AM12.7 (VEE), AM12.8 (VSS), AM13.6 (Inh), AM13.7 (VEE), AM13.8 (VSS), J1.G, J1.S, J2.S, RV1.3, RV10.3, RV11.3, RV12.3, RV2.3, RV3.3, RV4.3, RV5.3, RV6.3, RV7.3, RV8.3, RV9.3, SW3.C, SW3.S2, SW4.C, SW4.S2, SW5.C, SW5.S2; no longer AM1.12 (X3), AM3.2 (X6), AM5.15 (X2)
- net HE1: now also AM1.1 (X4), AM11.1 (X4); no longer AM3.15 (X2)
- net HE17: now also AM3.1 (X4); no longer AM3.14 (X1)
- net HE18: now also AM3.2 (X6); no longer AM3.13 (X0)
- net HE19: now also AM3.4 (X7); no longer AM3.12 (X3)
- net HE2: now also AM1.2 (X6), AM11.2 (X6); no longer AM1.15 (X2)
- net HE20: now also AM3.5 (X5); no longer AM3.1 (X4)
- net HE21: now also AM3.15 (X2); no longer AM3.4 (X7)
- net HE22: now also AM3.14 (X1); no longer AM3.5 (X5)
- net HE23: now also AM3.13 (X0); no longer AM4.1 (X4)
- net HE24: now also AM3.12 (X3); no longer AM4.2 (X6)
- net HE25: now also AM4.1 (X4); no longer AM4.4 (X7)
- net HE26: now also AM4.2 (X6); no longer AM4.5 (X5)
- net HE27: now also AM4.4 (X7); no longer AM4.15 (X2)
- net HE28: now also AM4.5 (X5); no longer AM4.14 (X1)
- net HE29: now also AM4.15 (X2); no longer AM4.13 (X0)
- net HE3: now also AM1.4 (X7), AM11.4 (X7); no longer AM1.14 (X1)
- net HE30: now also AM4.14 (X1); no longer AM4.12 (X3)
- net HE31: now also AM4.13 (X0); no longer AM7.1 (X4)
- net HE32: now also AM4.12 (X3); no longer AM5.1 (X4)
- net HE33: now also AM5.1 (X4); no longer AM5.2 (X6)
- net HE34: now also AM5.2 (X6); no longer AM5.4 (X7)
- net HE35: now also AM5.4 (X7); no longer AM5.5 (X5)
- net HE36: now also AM5.5 (X5); no longer AM5.14 (X1)
- net HE37: now also AM5.15 (X2); no longer AM5.13 (X0)
- net HE38: now also AM5.14 (X1); no longer AM5.12 (X3)
- net HE39: now also AM5.13 (X0); no longer AM6.1 (X4)
- net HE4: now also AM1.5 (X5), AM11.5 (X5); no longer AM1.13 (X0)
- net HE40: now also AM5.12 (X3); no longer AM6.2 (X6)
- net HE41: now also AM6.1 (X4); no longer AM6.4 (X7)
- net HE42: now also AM6.2 (X6); no longer AM6.5 (X5)
- net HE43: now also AM6.4 (X7); no longer AM6.15 (X2)
- net HE44: now also AM6.5 (X5); no longer AM7.2 (X6)
- net HE45: now also AM6.15 (X2); no longer AM7.4 (X7)
- net HE46: now also AM6.14 (X1); no longer AM7.5 (X5)
- net HE47: now also AM6.13 (X0); no longer AM8.1 (X4)
- net HE48: now also AM6.12 (X3); no longer AM8.2 (X6)
- net HE49: now also AM7.1 (X4); no longer AM8.4 (X7)
- net HE5: now also AM1.15 (X2), AM11.15 (X2); no longer AM1.1 (X4)
- net HE50: no longer AM8.5 (X5)
- net HE55: no longer AM6.12 (X3)
- net HE56: no longer AM6.13 (X0)
- net HE57: no longer AM6.14 (X1)
- net HE58: no longer AM7.15 (X2)
- net HE59: no longer AM7.14 (X1)
- net HE6: now also AM1.14 (X1), AM11.14 (X1); no longer AM1.2 (X6)
- net HE60: no longer AM7.13 (X0)
- net HE61: no longer AM7.12 (X3)
- net HE62: no longer AM8.12 (X3)
- net HE63: no longer AM8.13 (X0)
- net HE64: no longer AM8.14 (X1)
- net HE65: no longer AM8.15 (X2)
- net HE7: now also AM1.13 (X0), AM11.13 (X0); no longer AM1.4 (X7)
- net HE8: now also AM1.12 (X3), AM11.12 (X3); no longer AM1.5 (X5)
- net MUX_OUT_10: now also AM11.3 (X)
- net MUX_SELECT_0: now also AM12.11 (A), AM13.11 (A)
- net MUX_SELECT_1: now also AM12.10 (B), AM13.10 (B)
- net MUX_SELECT_2: now also AM12.9 (C), AM13.9 (C)
- net ENCODER_3_A: now reaches A1.10 (SPI1_POCI)
- net ENCODER_3_A: now also SW5.A
- net ENCODER_3_B: now reaches A1.11 (SPI1_PICO)
- net ENCODER_3_B: now also SW5.B
- net Audio_in_1: now reaches A1.16 (AUDIO_IN_1)
- net Audio_in_1: now also J1.T
- net Audio_in_2: now reaches A1.17 (AUDIO_IN_2)
- net Audio_in_2: now also J1.R
- net Audio_out_1: now reaches A1.18 (AUDIO_OUT_1)
- net Audio_out_1: now also J2.T
- net Audio_out_2: now reaches A1.19 (AUDIO_OUT_2)
- net Audio_out_2: now also J2.R
- net ENB_B: now reaches A1.3 (SD_DATA_2)
- net ENCODER_1_Btn: now reaches A1.33 (SAI2_SD_A)
- net ENCODER_1_Btn: now also SW3.S1
- net ENCODER_2_Btn: now reaches A1.34 (SAI2_FS)
- net ENCODER_2_Btn: now also SW4.S1
- net ENCODER_3_Btn: now reaches A1.36 (USB_D_-)
- net ENCODER_3_Btn: now also SW5.S1
- net ENB_A: now reaches A1.4 (SD_DATA_1)
- net ENCODER_1_A: now reaches A1.6 (SD_CMD)
- net ENCODER_1_A: now also SW3.A
- net ENCODER_1_B: now reaches A1.7 (SD_CLK)
- net ENCODER_1_B: now also SW3.B
- net ENCODER_2_A: now reaches A1.8 (SPI1_CS)
- net ENCODER_2_A: now also SW4.A
- net ENCODER_2_B: now reaches A1.9 (SPI1_SCK)
- net ENCODER_2_B: now also SW4.B
- net MUX_OUT_11 renamed MUX_OUT_12
- net MUX_OUT_12: now also AM12.3 (X), AM13.3 (X); no longer AM11.3 (X)
- new net: D2.2 (A), R2.1
- new net: D3.2 (A), R3.1
- new net: D1.2 (A), R1.1
- new net POT1: RV1.2
- new net POT10: RV10.2
- new net POT11: RV11.2
- new net POT12: RV12.2
- new net POT2: RV2.2
- new net POT3: RV3.2
- new net POT4: RV4.2
- new net POT5: RV5.2
- new net POT6: RV6.2
- new net POT7: RV7.2
- new net POT8: RV8.2
- new net POT9: RV9.2
- no-connect marks 41 -> 0
Other:
- moved on the sheet: A1, AM1, AM10, AM11, AM2, AM3, AM4, AM5, AM6, AM7, AM8, AM9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

Commit message: add pins for screen
Parts:
- added J3: Screen Connector, Connector_PinHeader_2.54mm:PinHeader_1x04_P2.54mm_Vertical, symbol Connector:Conn_01x04_Socket
Other:
- note added: "AM1"
- note added: "AM10"
- note added: "AM11"
- note added: "AM12"
- note added: "AM13"
- note added: "AM14"
- note added: "AM15"
- note added: "AM2"
- note added: "AM3"
- note added: "AM4"
- note added: "AM5"
- note added: "AM6"
- note added: "AM7"
- note added: "AM8"
- note added: "AM9"
- moved on the sheet: A1, AM1, AM10, AM11, AM12, AM13, AM2, AM3, AM4, AM5, AM6, AM7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

Commit message: Update keyboard_keyboard.kicad_sch
Parts:
- removed SW3, SW4, SW5: RotaryEncoder_Switch, Rotary_Encoder:RotaryEncoder_Alps_EC11E_Vertical_H20mm, symbol Device:RotaryEncoder_Switch
Connections:
- net +3.3VA: now also J3.1 (Pin_1)
- net GND: now also J3.2 (Pin_2)
- net HE1: no longer AM11.1 (X4)
- net HE10: no longer AM2.2 (X6)
- net HE11: no longer AM2.4 (X7)
- net HE12: no longer AM2.5 (X5)
- net HE13: no longer AM2.15 (X2)
- net HE14: no longer AM2.14 (X1)
- net HE15: no longer AM2.13 (X0)
- net HE16: no longer AM2.12 (X3)
- net HE17: no longer AM3.1 (X4)
- net HE18: no longer AM3.2 (X6)
- net HE19: no longer AM3.4 (X7)
- net HE2: no longer AM11.2 (X6)
- net HE20: no longer AM3.5 (X5)
- net HE21: no longer AM3.15 (X2)
- net HE22: no longer AM3.14 (X1)
- net HE23: no longer AM3.13 (X0)
- net HE24: no longer AM3.12 (X3)
- net HE25: no longer AM4.1 (X4)
- net HE26: no longer AM4.2 (X6)
- net HE27: no longer AM4.4 (X7)
- net HE28: no longer AM4.5 (X5)
- net HE29: no longer AM4.15 (X2)
- net HE3: no longer AM11.4 (X7)
- net HE30: no longer AM4.14 (X1)
- net HE31: no longer AM4.13 (X0)
- net HE32: no longer AM4.12 (X3)
- net HE33: no longer AM5.1 (X4)
- net HE34: no longer AM5.2 (X6)
- net HE35: no longer AM5.4 (X7)
- net HE36: no longer AM5.5 (X5)
- net HE37: no longer AM5.15 (X2)
- net HE38: no longer AM5.14 (X1)
- net HE39: no longer AM5.13 (X0)
- net HE4: no longer AM11.5 (X5)
- net HE40: no longer AM5.12 (X3)
- net HE41: no longer AM6.1 (X4)
- net HE42: no longer AM6.2 (X6)
- net HE43: no longer AM6.4 (X7)
- net HE44: no longer AM6.5 (X5)
- net HE45: no longer AM6.15 (X2)
- net HE46: no longer AM6.14 (X1)
- net HE47: no longer AM6.13 (X0)
- net HE48: no longer AM6.12 (X3)
- net HE49: no longer AM7.1 (X4)
- net HE5: no longer AM11.15 (X2)
- net HE51: no longer AM9.1 (X4)
- net HE52: no longer AM9.2 (X6)
- net HE53: no longer AM9.4 (X7)
- net HE54: no longer AM9.5 (X5)
- net HE6: no longer AM11.14 (X1)
- net HE66: no longer AM9.12 (X3)
- net HE67: no longer AM9.13 (X0)
- net HE68: no longer AM9.14 (X1)
- net HE69: no longer AM9.15 (X2)
- net HE7: no longer AM11.13 (X0)
- net HE70: no longer AM10.12 (X3)
- net HE71: no longer AM10.15 (X2)
- net HE72: no longer AM10.14 (X1)
- net HE73: no longer AM10.13 (X0)
- net HE74: no longer AM10.1 (X4)
- net HE75: no longer AM10.2 (X6)
- net HE76: no longer AM10.4 (X7)
- net HE77: no longer AM10.5 (X5)
- net HE8: no longer AM11.12 (X3)
- net HE9: no longer AM2.1 (X4)
- net SDA: now reaches J3.3 (Pin_3)
- net SDA: now also A1.13 (I2C1_SDA)
- net SCL: now reaches J3.4 (Pin_4)
- net SCL: now also A1.12 (I2C1_SCL)
- net ENB_C: now reaches A1.2 (SD_DATA_3)
- net ENCODER_1_A: no longer names the net of A1.6 (SD_CMD)
- net ENCODER_1_B: no longer names the net of A1.7 (SD_CLK)
- net ENCODER_1_Btn renamed MUX_OUT_14
- net ENCODER_2_A: no longer names the net of A1.8 (SPI1_CS)
- net ENCODER_2_B: no longer names the net of A1.9 (SPI1_SCK)
- net ENCODER_2_Btn: no longer names the net of A1.34 (SAI2_FS)
- net ENCODER_3_A: no longer names the net of A1.10 (SPI1_POCI)
- net ENCODER_3_B: no longer names the net of A1.11 (SPI1_PICO)
- net ENCODER_3_Btn: no longer names the net of A1.36 (USB_D_-)
Other:
- moved on the sheet: AM10, AM8, AM9, C146, C147, C161

Commit message: Update keyboard_keyboard.kicad_sch
Parts:
- added AM14, AM15: SN74LV4051A, Package_SO:TSSOP-16_4.4x5mm_P0.65mm, symbol 4xxx:4051
- added C150, C151: 100n, Capacitor_SMD:C_0402_1005Metric, symbol Device:C
- added U1: 74HC138, symbol 74xx:74HC138
Connections:
- net +3.3VA: now also A1.38 (3V3_D), AM14.16 (VDD), AM15.16 (VDD), C150.1, C151.1, U1.5 (~{E1}), U1.6 (E2)
- net ENB_A: now also U1.1 (A0)
- net ENB_B: now also U1.2 (A1)
- net ENB_C: now also U1.3 (A2)
- net GND: now also A1.20 (AGND), A1.40 (DGND), AM10.12 (X3), AM11.12 (X3), AM8.12 (X3), AM8.13 (X0), AM14.7 (VEE), AM14.8 (VSS), AM15.12 (X3), AM15.13 (X0), AM15.14 (X1), AM15.15 (X2), AM15.7 (VEE), AM15.8 (VSS), C150.2, C151.2, U1.4 (~{E0}), U1.8 (GND); no longer AM10.6 (Inh), AM11.6 (Inh), AM12.6 (Inh), AM13.6 (Inh)
- net HE10: now also AM2.2 (X6)
- net HE100: now also AM13.12 (X3)
- net HE11: now also AM2.4 (X7)
- net HE12: now also AM2.5 (X5)
- net HE13: now also AM2.15 (X2)
- net HE14: now also AM2.14 (X1)
- net HE15: now also AM3.1 (X4)
- net HE16: now also AM3.2 (X6)
- net HE17: now also AM3.4 (X7)
- net HE18: now also AM3.5 (X5)
- net HE19: now also AM3.15 (X2)
- net HE20: now also AM3.14 (X1)
- net HE21: now also AM3.13 (X0)
- net HE22: now also AM3.12 (X3)
- net HE23: now also AM4.1 (X4)
- net HE24: now also AM4.2 (X6)
- net HE25: now also AM4.4 (X7)
- net HE26: now also AM4.5 (X5)
- net HE27: now also AM4.15 (X2)
- net HE28: now also AM2.13 (X0)
- net HE29: now also AM2.12 (X3)
- net HE30: now also AM5.1 (X4)
- net HE31: now also AM5.2 (X6)
- net HE32: now also AM5.4 (X7)
- net HE33: now also AM5.5 (X5)
- net HE34: now also AM5.15 (X2)
- net HE35: now also AM5.14 (X1)
- net HE36: now also AM5.13 (X0)
- net HE37: now also AM5.12 (X3)
- net HE38: now also AM6.1 (X4)
- net HE39: now also AM6.2 (X6)
- net HE40: now also AM6.4 (X7)
- net HE41: now also AM4.14 (X1)
- net HE42: now also AM4.13 (X0)
- net HE43: now also AM4.12 (X3)
- net HE44: now also AM7.1 (X4)
- net HE45: now also AM7.2 (X6)
- net HE46: now also AM7.4 (X7)
- net HE47: now also AM7.5 (X5)
- net HE48: now also AM7.15 (X2)
- net HE49: now also AM7.14 (X1)
- net HE50: now also AM7.13 (X0)
- net HE51: now also AM7.12 (X3)
- net HE52: now also AM8.1 (X4)
- net HE53: now also AM8.2 (X6)
- net HE54: now also AM6.5 (X5)
- net HE55: now also AM6.15 (X2)
- net HE56: now also AM6.14 (X1)
- net HE57: now also AM6.13 (X0)
- net HE58: now also AM6.12 (X3)
- net HE59: now also AM9.1 (X4)
- net HE60: now also AM9.2 (X6)
- net HE61: now also AM9.4 (X7)
- net HE62: now also AM9.5 (X5)
- net HE63: now also AM9.15 (X2)
- net HE64: now also AM9.14 (X1)
- net HE65: now also AM9.13 (X0)
- net HE66: now also AM9.12 (X3)
- net HE67: now also AM8.4 (X7)
- net HE68: now also AM8.5 (X5)
- net HE69: now also AM8.15 (X2)
- net HE70: now also AM8.14 (X1)
- net HE71: now also AM10.1 (X4)
- net HE72: now also AM10.2 (X6)
- net HE73: now also AM10.4 (X7)
- net HE74: now also AM11.1 (X4)
- net HE75: now also AM11.2 (X6)
- net HE76: now also AM11.4 (X7)
- net HE77: now also AM11.5 (X5)
- net HE78: now also AM11.15 (X2)
- net HE79: now also AM11.14 (X1)
- net HE80: now also AM11.13 (X0)
- net HE81: now also AM10.5 (X5)
- net HE82: now also AM10.15 (X2)
- net HE83: now also AM10.14 (X1)
- net HE84: now also AM10.13 (X0)
- net HE85: now also AM12.1 (X4)
- net HE86: now also AM12.2 (X6)
- net HE87: now also AM12.4 (X7)
- net HE88: now also AM12.5 (X5)
- net HE89: now also AM12.15 (X2)
- net HE9: now also AM2.1 (X4)
- net HE90: now also AM12.14 (X1)
- net HE91: now also AM12.13 (X0)
- net HE92: now also AM12.12 (X3)
- net HE93: now also AM13.1 (X4)
- net HE94: now also AM13.2 (X6)
- net HE95: now also AM13.4 (X7)
- net HE96: now also AM13.5 (X5)
- net HE97: now also AM13.15 (X2)
- net HE98: now also AM13.14 (X1)
- net HE99: now also AM13.13 (X0)
- net MUX_OUT_14: now also AM14.3 (X), AM15.3 (X)
- net MUX_SELECT_0: now also A1.8 (SPI1_CS), AM14.11 (A), AM15.11 (A)
- net MUX_SELECT_1: now also A1.9 (SPI1_SCK), AM14.10 (B), AM15.10 (B)
- net MUX_SELECT_2: now also A1.10 (SPI1_POCI), AM14.9 (C), AM15.9 (C)
- net POT1: now also AM14.1 (X4)
- net POT10: now also AM15.2 (X6)
- net POT11: now also AM15.4 (X7)
- net POT12: now also AM15.5 (X5)
- net POT2: now also AM14.2 (X6)
- net POT3: now also AM14.4 (X7)
- net POT4: now also AM14.5 (X5)
- net POT5: now also AM14.15 (X2)
- net POT6: now also AM14.14 (X1)
- net POT7: now also AM14.13 (X0)
- net POT8: now also AM14.12 (X3)
- net POT9: now also AM15.1 (X4)
- new net ENABLE_10: AM10.6 (Inh), U1.15 (~{Y0})
- new net ENABLE_11: AM11.6 (Inh), U1.14 (~{Y1})
- new net ENABLE_12: AM12.6 (Inh), U1.13 (~{Y2})
- new net ENABLE_13: AM13.6 (Inh), U1.12 (~{Y3})
- new net ENABLE_14: AM14.6 (Inh), U1.11 (~{Y4})
- new net ENABLE_15: AM15.6 (Inh), U1.10 (~{Y5})
Other:
- moved on the sheet: A1, AM1, AM10, AM11, AM12, AM13, AM2, AM3, AM4, AM5, AM6, AM7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

Commit message: update wires
Connections:
- net HE28: now also AM2.12 (X3); no longer AM2.13 (X0)
- net HE29: now also AM2.13 (X0); no longer AM2.12 (X3)
- net HE86: no longer C198.1, HE87.2 (OUT)
- net HE87: now also C198.1, HE87.2 (OUT)
Other:
- moved on the sheet: AM10, AM11, AM12, AM13, AM14, AM15, AM8, AM9, C146, C147, C148, C149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
