File: keyboard_keyboard/kicad/keyboard_keyboard.kicad_sch (KiCad schematic)
At the start: 464 parts, among them J1 AudioJack3_Ground, J2 AudioJack3_Ground, J3 Screen Connector, J4 DIN-5, J5 DIN-5, J6 Conn_01x04_Socket, J7 Conn_01x04_Socket, U1 74HC138, U2 6N138

Commit message: Add vibrato on/off toggle & increase dead zone
- Add VIBRATO_SETTING menu item to enable/disable vibrato via CC1 (off by default)
- Increase VIBRATO_DEAD_ZONE from 30 to 100 to prevent accidental triggering
- Display vibrato as ON/OFF instead of numeric value in settings menu
- Only send vibrato CC1 when enabled and settings menu is closed
- Fix Embed.toml chip identifier to "STM32H750VBTx"
- Add LM317L linear regulator circuit to schematic for clean 3.3V rail
- Update .gitignore to exclude KiCad temporary files
Parts:
- added C152: 1uf, symbol Device:C_Polarized
- added C153: 220uf, symbol Device:C_Polarized
- added C1_: 0.1uf, symbol Device:C
- added R10: 33, symbol Device:R_US
- added R1_: 330, symbol Device:R_US
- added R2_: 220, symbol Device:R_US
- added U3: LM317T, Package_TO_SOT_SMD:SOT-89-3, symbol Regulator_Linear:LM317L_SOT-89
Connections:
- net GND: now also C152.2, C153.2, C1_.2, R10.2
- new net: R1_.1, R2_.2, U3.1 (ADJ)
- new net: R10.1, R1_.2
- new net 5v: C1_.1, U3.3 (VI)
- new net vout: C152.1, C153.1, R2_.1, U3.2 (VO)
