File: keyboard_keyboard/kicad/keyboard_keyboard.kicad_pcb (KiCad board)
At the start: 2 copper layers, 447.8 x 353.1 mm, 484 parts, among them J1 Conn_01x30, J1 TYPE-C-31-M-12, J2 JST_SH, SW1 TS-1187A-B-A-B, SW2 TS-1187A-B-A-B, U1 USBLC6-2SC6, U2 TLV75733PDBV, U3 XC6206P332MR-G, U4 AT32F405RCT7, Y1 X322512MSB4SI

Commit message: move things around
Parts:
- removed C29: 100n, Capacitor_SMD:C_0402_1005Metric
- removed C30: 4.7n, Capacitor_SMD:C_0402_1005Metric
- removed HE15: MT9102ET, Package_TO_SOT_SMD:SOT-23-3
- removed MX086: MX-NoLED, MX_Only:MXOnly-1.5U-Hotswap
- removed the MX43 at (263.8, 47.1)
- moved MX36 449.9 mm to (250.4, -272.9)
- moved C31 401.1 mm to (9.62, -294.3)
- moved C32 401.1 mm to (14.8, -294.3)
- moved HE16 401.1 mm to (12.2, -293.5)
- moved MX16 401.1 mm to (12.2, -293.5)
- moved C27 323.5 mm to (271.6, -314.8)
- moved C28 323.5 mm to (276.8, -314.8)
- moved HE14 323.5 mm to (274.2, -314.0)
- moved MX14 323.5 mm to (274.2, -314.0)
- moved AM2 323.4 mm to (192.8, -303.4)
- moved AM1 323.3 mm to (78.4, -303.8)
- moved C5 323.3 mm to (57.2, -314.8)
- moved C6 323.3 mm to (62.4, -314.8)
- moved HE3 323.3 mm to (59.8, -314.0)
- moved MX3 323.3 mm to (59.8, -314.0)
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Routing:
- net VBUS: vias 2 -> 0
- net NRST: vias 2 -> 0
- net MUX_SELECT_2: vias 10 -> 0
- net MUX_SELECT_1: vias 10 -> 0
- net MUX_SELECT_0: vias 10 -> 0
- net MUX_OUT_9: vias 2 -> 0
- net MUX_OUT_8: vias 2 -> 0
- net MUX_OUT_7: vias 2 -> 0
- net MUX_OUT_4: vias 2 -> 0
- net MUX_OUT_3: vias 2 -> 0
- net MUX_OUT_2: vias 2 -> 0
- net MUX_OUT_1: vias 2 -> 0
- net HE1: vias 2 -> 0
- net GND: vias 638 -> 62
- net BOOT0: vias 2 -> 0
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
Commit message: more routing
Parts:
- removed MX44: 2.25U, HE60:MX-2.25U
- removed MX55: 1.75U, HE60:MX-1.75U
- removed MX56: 2.75U, HE60:MX-2.75U
- removed MX58, MX60, MX62, MX70, MX72, MX74, MX76: 1.25U, HE60:MX-1.25U
- removed MX59, MX63, MX71, MX75: 1.5U, HE60:MX-1.5U
- removed MX65: 2.25U, HE60:MX-2.25U-ReversedStabilizers
- removed the MX66 at (130.4, 85.2)
- removed the MX67 at (142.3, 85.2)
- removed the MX68 at (163.8, 85.2)
- removed MX69, MX73: 1U, HE60:MX-1U
- added MX45: 1U, HE60:MX-1U, F.Cu at (202.7, -252.3)
- added MX45: 1U, HE60:MX-1U, F.Cu at (221.8, -252.3)
- added MX45: 1U, HE60:MX-1U, F.Cu at (274.2, -272.9)
- added MX61: 1U, HE60:MX-1U, F.Cu at (259.9, -252.4)
- added MX61: 1U, HE60:MX-1U, F.Cu at (78.9, -231.8)
- added MX61: 1U, HE60:MX-1U, F.Cu at (136.0, -231.8)
- added MX61: 1U, HE60:MX-1U, F.Cu at (17.0, -231.8)
- added MX61: 1U, HE60:MX-1U, F.Cu at (97.9, -231.8)
- added MX61: 1U, HE60:MX-1U, F.Cu at (155.1, -231.8)
- added MX61: 1U, HE60:MX-1U, F.Cu at (212.3, -231.8)
- added MX61: 1U, HE60:MX-1U, F.Cu at (174.1, -231.8)
- added MX61: 1U, HE60:MX-1U, F.Cu at (193.2, -231.8)
- added MX61: 1U, HE60:MX-1U, F.Cu at (117.0, -231.8)
- moved TH2 460.8 mm to (-26.0, -249.9)
- moved HE44 423.2 mm to (274.2, -272.9)
- moved C87 423.2 mm to (271.6, -273.7)
- moved C88 423.2 mm to (276.8, -273.7)
- moved HE58 418.4 mm to (259.9, -252.3)
- moved C115 418.4 mm to (262.9, -250.7)
- moved C116 418.4 mm to (256.9, -250.7)
- moved HE59 415.9 mm to (279.1, -252.6)
- moved C117 415.7 mm to (282.2, -250.7)
- moved C118 414.9 mm to (274.7, -250.7)
- moved MX61 414.9 mm to (278.9, -252.3)
- moved C137 322.6 mm to (215.3, -230.2)
- moved C138 322.6 mm to (209.3, -230.2)
- moved HE69 322.6 mm to (212.3, -231.8)
- moved C110 321.9 mm to (199.7, -250.7)
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
Commit message: more keys
Parts:
- removed the C125 at (-158.9, 6.10)
- removed the C127 at (-147.0, 6.10)
- removed the C128 at (-153.0, 6.10)
- removed the C155 at (24.0, -277.7)
- removed the C155 at (-129.0, -123.0)
- removed the C59 at (-138.8, -74.8)
- removed the C60 at (-133.6, -74.8)
- removed the C61 at (-137.1, -119.1)
- removed the C62 at (-131.9, -119.1)
- removed the C71 at (-127.9, 46.9)
- removed the C72 at (-135.6, 39.8)
- removed the C85 at (-132.1, -97.1)
- removed the C86 at (-126.9, -97.1)
- removed the HE30 at (-136.2, -74.0)
- removed the HE31 at (-134.5, -118.3)
- removed the HE36 at (-138.2, 40.6)
- removed the HE43 at (-129.5, -96.3)
- removed the HE64 at (-150.0, 4.50)
- removed the MX30 at (-136.2, -74.0)
- removed the MX31 at (-134.5, -118.3)
- removed the MX36 at (250.4, -272.9)
- removed the MX45 at (202.7, -252.3)
- removed the MX45 at (221.8, -252.3)
- removed the MX45 at (274.2, -272.9)
- removed the MX61 at (259.9, -252.4)
- removed the MX61 at (78.9, -231.8)
- removed the MX61 at (136.0, -231.8)
- removed the MX61 at (17.0, -231.8)
- removed the MX61 at (97.9, -231.8)
- removed the MX61 at (155.1, -231.8)
- removed the MX61 at (212.3, -231.8)
- removed the MX61 at (174.1, -231.8)
- removed the MX61 at (278.9, -252.3)
- removed the MX61 at (193.2, -231.8)
- removed the MX61 at (117.0, -231.8)
- removed the R3 at (23.8, -273.4)
- removed the R3 at (-127.6, -118.8)
- removed SWR3: RotaryEncoder_Switch, Keebio-Parts:RotaryEncoder_EC11_Nonplated
- added A1: Electrosmith_Daisy_Seed_Rev4, Module:Electrosmith_Daisy_Seed, F.Cu at (384.8, -198.3)
- added AM10: SN74LV4051A, Package_SO:TSSOP-16_4.4x5mm_P0.65mm, B.Cu at (347.1, -266.3)
- added AM11: SN74LV4051A, Package_SO:TSSOP-16_4.4x5mm_P0.65mm, B.Cu at (347.1, -272.9)
- added C155: 100n, Capacitor_SMD:C_0402_1005Metric, B.Cu at (214.3, -268.9)
- added C161: 100n, Capacitor_SMD:C_0402_1005Metric, B.Cu at (293.2, -262.9)
- added C162: 100n, Capacitor_SMD:C_0402_1005Metric, B.Cu at (293.2, -264.9)
- added C163: 100n, Capacitor_SMD:C_0402_1005Metric, B.Cu at (243.8, -60.1)
- added C164: 4.7n, Capacitor_SMD:C_0402_1005Metric, B.Cu at (238.6, -60.1)
- added C165: 100n, Capacitor_SMD:C_0402_1005Metric, B.Cu at (271.3, -142.2)
- added C166: 4.7n, Capacitor_SMD:C_0402_1005Metric, B.Cu at (276.5, -142.2)
- added C167: 100n, Capacitor_SMD:C_0402_1005Metric, B.Cu at (290.3, -142.2)
- added C168: 4.7n, Capacitor_SMD:C_0402_1005Metric, B.Cu at (295.5, -142.2)
- added C169: 100n, Capacitor_SMD:C_0402_1005Metric, B.Cu at (296.1, -258.9)
- added C170: 4.7n, Capacitor_SMD:C_0402_1005Metric, B.Cu at (296.1, -260.9)
- added C171: 100n, Capacitor_SMD:C_0402_1005Metric, B.Cu at (296.1, -262.9)
- added C172: 4.7n, Capacitor_SMD:C_0402_1005Metric, B.Cu at (296.1, -264.9)
- added C173: 100n, Capacitor_SMD:C_0402_1005Metric, B.Cu at (296.1, -266.8)
- added C174: 4.7n, Capacitor_SMD:C_0402_1005Metric, B.Cu at (296.1, -268.8)
- added C175: 100n, Capacitor_SMD:C_0402_1005Metric, B.Cu at (296.1, -270.8)
- added C176: 4.7n, Capacitor_SMD:C_0402_1005Metric, B.Cu at (296.1, -272.7)
- added C177: 100n, Capacitor_SMD:C_0402_1005Metric, B.Cu at (296.1, -274.7)
- added C178: 4.7n, Capacitor_SMD:C_0402_1005Metric, B.Cu at (296.1, -276.7)
- added C179: 100n, Capacitor_SMD:C_0402_1005Metric, B.Cu at (299.0, -258.9)
- added C180: 4.7n, Capacitor_SMD:C_0402_1005Metric, B.Cu at (299.0, -260.9)
- added C181: 100n, Capacitor_SMD:C_0402_1005Metric, B.Cu at (299.0, -262.9)
- added C182: 4.7n, Capacitor_SMD:C_0402_1005Metric, B.Cu at (299.0, -264.9)
- added C183: 100n, Capacitor_SMD:C_0402_1005Metric, B.Cu at (299.0, -266.8)
- added C184: 4.7n, Capacitor_SMD:C_0402_1005Metric, B.Cu at (299.0, -268.8)
- added C185: 100n, Capacitor_SMD:C_0402_1005Metric, B.Cu at (299.0, -270.8)
- added C186: 4.7n, Capacitor_SMD:C_0402_1005Metric, B.Cu at (299.0, -272.7)
- added C187: 100n, Capacitor_SMD:C_0402_1005Metric, B.Cu at (299.0, -274.7)
- added C188: 4.7n, Capacitor_SMD:C_0402_1005Metric, B.Cu at (299.0, -276.7)
- added C189: 100n, Capacitor_SMD:C_0402_1005Metric, B.Cu at (301.9, -258.9)
- added C190: 4.7n, Capacitor_SMD:C_0402_1005Metric, B.Cu at (301.9, -260.9)
- added C191: 100n, Capacitor_SMD:C_0402_1005Metric, B.Cu at (301.9, -262.9)
- added C192: 4.7n, Capacitor_SMD:C_0402_1005Metric, B.Cu at (301.9, -264.9)
- added C193: 100n, Capacitor_SMD:C_0402_1005Metric, B.Cu at (301.9, -266.8)
- added C194: 4.7n, Capacitor_SMD:C_0402_1005Metric, B.Cu at (301.9, -268.8)
- added C195: 100n, Capacitor_SMD:C_0402_1005Metric, B.Cu at (301.9, -270.8)
- added C196: 4.7n, Capacitor_SMD:C_0402_1005Metric, B.Cu at (301.9, -272.7)
- added C197: 100n, Capacitor_SMD:C_0402_1005Metric, B.Cu at (301.9, -274.7)
- added C198: 4.7n, Capacitor_SMD:C_0402_1005Metric, B.Cu at (301.9, -276.7)
- added C199: 100n, Capacitor_SMD:C_0402_1005Metric, B.Cu at (304.7, -258.9)
- added C200: 4.7n, Capacitor_SMD:C_0402_1005Metric, B.Cu at (304.7, -260.9)
- added C201: 100n, Capacitor_SMD:C_0402_1005Metric, B.Cu at (304.7, -262.9)
- added C202: 4.7n, Capacitor_SMD:C_0402_1005Metric, B.Cu at (304.7, -264.9)
- added C203: 100n, Capacitor_SMD:C_0402_1005Metric, B.Cu at (304.7, -266.8)
- added C204: 4.7n, Capacitor_SMD:C_0402_1005Metric, B.Cu at (304.7, -268.8)
- added C205: 100n, Capacitor_SMD:C_0402_1005Metric, B.Cu at (304.7, -270.8)
- added C206: 4.7n, Capacitor_SMD:C_0402_1005Metric, B.Cu at (304.7, -272.7)
- added C207: 100n, Capacitor_SMD:C_0402_1005Metric, B.Cu at (304.7, -274.7)
- added C208: 4.7n, Capacitor_SMD:C_0402_1005Metric, B.Cu at (304.7, -276.7)
- added C209: 100n, Capacitor_SMD:C_0402_1005Metric, B.Cu at (307.6, -258.9)
- added C210: 4.7n, Capacitor_SMD:C_0402_1005Metric, B.Cu at (307.6, -260.9)
- added C211: 100n, Capacitor_SMD:C_0402_1005Metric, B.Cu at (307.6, -262.9)
- added C212: 4.7n, Capacitor_SMD:C_0402_1005Metric, B.Cu at (307.6, -264.9)
- added C213: 100n, Capacitor_SMD:C_0402_1005Metric, B.Cu at (307.6, -266.8)
- added C214: 4.7n, Capacitor_SMD:C_0402_1005Metric, B.Cu at (307.6, -268.8)
- added C215: 100n, Capacitor_SMD:C_0402_1005Metric, B.Cu at (307.6, -270.8)
- added C216: 4.7n, Capacitor_SMD:C_0402_1005Metric, B.Cu at (307.6, -272.7)
- added C217: 100n, Capacitor_SMD:C_0402_1005Metric, B.Cu at (307.6, -274.7)
- added C218: 4.7n, Capacitor_SMD:C_0402_1005Metric, B.Cu at (307.6, -276.7)
- added C219: 100n, Capacitor_SMD:C_0402_1005Metric, B.Cu at (310.5, -258.9)
- added C220: 4.7n, Capacitor_SMD:C_0402_1005Metric, B.Cu at (310.5, -260.9)
- added C221: 100n, Capacitor_SMD:C_0402_1005Metric, B.Cu at (310.5, -262.9)
- added C222: 4.7n, Capacitor_SMD:C_0402_1005Metric, B.Cu at (310.5, -264.9)
- added C223: 100n, Capacitor_SMD:C_0402_1005Metric, B.Cu at (310.5, -266.8)
- added C224: 4.7n, Capacitor_SMD:C_0402_1005Metric, B.Cu at (310.5, -268.8)
- added C225: 100n, Capacitor_SMD:C_0402_1005Metric, B.Cu at (310.5, -270.8)
- added C226: 4.7n, Capacitor_SMD:C_0402_1005Metric, B.Cu at (310.5, -272.7)
- added C29: 100n, Capacitor_SMD:C_0402_1005Metric, B.Cu at (-18.2, -121.6)
- added C30: 4.7n, Capacitor_SMD:C_0402_1005Metric, B.Cu at (-23.4, -121.6)
- added HE100: MT9102ET, Package_TO_SOT_SMD:SOT-23-3, B.Cu at (236.1, -310.4)
- added HE101: MT9102ET, Package_TO_SOT_SMD:SOT-23-3, B.Cu at (236.1, -315.1)
- added HE15: MT9102ET, Package_TO_SOT_SMD:SOT-23-3, B.Cu at (-20.8, -120.8)
- added HE70: MT9102ET, Package_TO_SOT_SMD:SOT-23-3, B.Cu at (241.2, -59.3)
- added HE71: MT9102ET, Package_TO_SOT_SMD:SOT-23-3, B.Cu at (273.9, -141.4)
- added HE72: MT9102ET, Package_TO_SOT_SMD:SOT-23-3, B.Cu at (292.9, -141.4)
- added HE73: MT9102ET, Package_TO_SOT_SMD:SOT-23-3, B.Cu at (182.8, -251.2)
- added HE74: MT9102ET, Package_TO_SOT_SMD:SOT-23-3, B.Cu at (215.5, -319.7)
- added HE75: MT9102ET, Package_TO_SOT_SMD:SOT-23-3, B.Cu at (215.5, -324.3)
- added HE76: MT9102ET, Package_TO_SOT_SMD:SOT-23-3, B.Cu at (220.6, -296.6)
- added HE77: MT9102ET, Package_TO_SOT_SMD:SOT-23-3, B.Cu at (220.6, -301.2)
- added HE78: MT9102ET, Package_TO_SOT_SMD:SOT-23-3, B.Cu at (220.6, -305.8)
- added HE79: MT9102ET, Package_TO_SOT_SMD:SOT-23-3, B.Cu at (220.6, -310.4)
- added HE80: MT9102ET, Package_TO_SOT_SMD:SOT-23-3, B.Cu at (220.6, -315.1)
- added HE81: MT9102ET, Package_TO_SOT_SMD:SOT-23-3, B.Cu at (220.6, -319.7)
- added HE82: MT9102ET, Package_TO_SOT_SMD:SOT-23-3, B.Cu at (220.6, -324.3)
- added HE83: MT9102ET, Package_TO_SOT_SMD:SOT-23-3, B.Cu at (225.8, -296.6)
- added HE84: MT9102ET, Package_TO_SOT_SMD:SOT-23-3, B.Cu at (225.8, -301.2)
- added HE85: MT9102ET, Package_TO_SOT_SMD:SOT-23-3, B.Cu at (225.8, -305.8)
- added HE86: MT9102ET, Package_TO_SOT_SMD:SOT-23-3, B.Cu at (225.8, -310.4)
- added HE87: MT9102ET, Package_TO_SOT_SMD:SOT-23-3, B.Cu at (225.8, -315.1)
- added HE88: MT9102ET, Package_TO_SOT_SMD:SOT-23-3, B.Cu at (225.8, -319.7)
- added HE89: MT9102ET, Package_TO_SOT_SMD:SOT-23-3, B.Cu at (225.8, -324.3)
- added HE90: MT9102ET, Package_TO_SOT_SMD:SOT-23-3, B.Cu at (230.9, -296.6)
- added HE91: MT9102ET, Package_TO_SOT_SMD:SOT-23-3, B.Cu at (230.9, -301.2)
- added HE92: MT9102ET, Package_TO_SOT_SMD:SOT-23-3, B.Cu at (230.9, -305.8)
- added HE93: MT9102ET, Package_TO_SOT_SMD:SOT-23-3, B.Cu at (230.9, -310.4)
- added HE94: MT9102ET, Package_TO_SOT_SMD:SOT-23-3, B.Cu at (230.9, -315.1)
- added HE95: MT9102ET, Package_TO_SOT_SMD:SOT-23-3, B.Cu at (230.9, -319.7)
- added HE96: MT9102ET, Package_TO_SOT_SMD:SOT-23-3, B.Cu at (230.9, -324.3)
- added HE97: MT9102ET, Package_TO_SOT_SMD:SOT-23-3, B.Cu at (236.1, -296.6)
- added HE98: MT9102ET, Package_TO_SOT_SMD:SOT-23-3, B.Cu at (236.1, -301.2)
- added HE99: MT9102ET, Package_TO_SOT_SMD:SOT-23-3, B.Cu at (236.1, -305.8)
- added MX44: 1u, HE60:MX-1U, F.Cu at (-20.7, -79.7)
- added MX55: 15U, HE60:MX-1U, F.Cu at (188.8, -79.7)
- added MX56: 1U, HE60:MX-1U, F.Cu at (207.9, -79.7)
- added MX58: 1U, HE60:MX-1U, F.Cu at (246.0, -79.7)
- added MX59: 1.5U, HE60:MX-1.5U, F.Cu at (-16.0, -59.1)
- added MX60: 1U, HE60:MX-1U, F.Cu at (26.9, -59.1)
- added MX61: 1U, HE60:MX-1U, F.Cu at (45.9, -59.1)
- added MX62: 1U, HE60:MX-1U, F.Cu at (65.0, -59.1)
- added MX63: 1U, HE60:MX-1U, F.Cu at (84.0, -59.1)
- added MX65: 1U, HE60:MX-1U, F.Cu at (122.2, -59.1)
- added MX69: 1U, HE60:MX-1U, F.Cu at (198.4, -59.1)
- added MX70: 1.5U, HE60:MX-1.5U, F.Cu at (241.2, -59.1)
- added MX71: 1U, HE60:MX-1U, F.Cu at (273.9, -141.4)
- added MX72: 1U, HE60:MX-1U, F.Cu at (292.9, -141.4)
- added MX73: 1U, HE60:MX-1U, F.Cu at (55.3, -242.2)
- added MX74: 1U, HE60:MX-1U, F.Cu at (15.0, -221.8)
- added MX75: 1U, HE60:MX-1U, F.Cu at (35.1, -221.9)
- added MX76: 1U, HE60:MX-1U, F.Cu at (55.5, -221.8)
- added PCB1: H60, HE60:H60, F.Cu at (179.8, -457.2)
- added R3: 12k, Resistor_SMD:R_0402_1005Metric, B.Cu at (218.3, -266.4)
- C145, C146, C148, C149, C150, C151, C152, C153, C154, C160, F1, J1, J2, R1, R2, R4, SW1, SW2, U1, U2, U3, U4, Y1: moved to F.Cu
- MX14: value 1U -> 1.5U; footprint HE60:MX-1U -> HE60:MX-1.5U
- MX15: value 2U -> 1U; footprint HE60:MX-2U -> HE60:MX-1U; moved to B.Cu
- MX17: value 1.5U -> 1U; footprint HE60:MX-1.5U -> HE60:MX-1U
- MX31: value 1.75U -> 1U; footprint HE60:MX-1.75U -> HE60:MX-1U
- MX43: value 2.25U -> 1.5U; footprint HE60:MX-2.25U -> HE60:MX-1.5U
- MX66: value 6.25U -> 1U; footprint HE60:MX-6.25U-ReversedStabilizers -> HE60:MX-1U
- MX67: value 7U -> 1U; footprint HE60:MX-7U-ReversedStabilizers -> HE60:MX-1U
- MX68: value 2.75U -> 1U; footprint HE60:MX-2.75U-ReversedStabilizers -> HE60:MX-1U
- TH2: moved to B.Cu
- moved H1 592.0 mm to (566.7, -353.8)
- moved H10 592.0 mm to (757.2, -312.8)
- moved H12 592.0 mm to (899.5, -312.8)
- moved H13 592.0 mm to (965.5, -312.7)
- moved H14 592.0 mm to (1003.7, -312.7)
- moved H15 592.0 mm to (569.1, -291.9)
- moved H16 592.0 mm to (633.4, -292.0)
- moved H17 592.0 mm to (709.6, -292.2)
- moved H18 592.0 mm to (785.8, -292.2)
- moved H19 592.0 mm to (861.4, -292.2)
- moved H2 592.0 mm to (642.9, -353.9)
- moved H20 592.0 mm to (927.4, -292.1)
- moved H21 592.0 mm to (569.1, -271.0)
- moved H22 592.0 mm to (638.2, -271.1)
- moved H23 592.0 mm to (714.4, -271.2)
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Routing:
- net GND: vias 62 -> 53
- net +3.3VA: vias 1 -> 3
- removed copper zone on B.Cu, net +3.3VA
- removed copper zone on B.Cu, net +5V
Other:
- board size 447.8 x 353.1 mm -> 1044 x 327.4 mm
- board text removed: "RESET"

Commit message: more keys
Parts:
- removed the CAP1 at (958.1, -340.6)
- removed the H1 at (566.7, -353.8)
- removed the H10 at (757.2, -312.8)
- removed the H11 at (833.4, -312.9)
- removed the H12 at (899.5, -312.8)
- removed the H13 at (965.5, -312.7)
- removed the H14 at (1003.7, -312.7)
- removed H15, H16, H17, H18: MountingHole, MountingHole:MountingHole_3mm
- removed the H19 at (861.4, -292.2)
- removed the H2 at (642.9, -353.9)
- removed the H20 at (927.4, -292.1)
- removed the H21 at (569.1, -271.0)
- removed the H22 at (638.2, -271.1)
- removed the H23 at (714.4, -271.2)
- removed the H24 at (790.6, -271.3)
- removed the H25 at (861.4, -271.2)
- removed the H26 at (899.5, -271.2)
- removed the H27 at (946.4, -271.1)
- removed the H28 at (1003.7, -271.0)
- removed the H29 at (609.6, -250.7)
- removed the H3 at (690.6, -354.0)
- removed the H30 at (685.8, -250.9)
- removed the H31 at (723.9, -250.9)
- removed the H32 at (800.1, -250.9)
- removed the H33 at (861.4, -250.9)
- removed the H34 at (927.4, -250.8)
- removed the H35 at (1003.7, -250.7)
- removed the H36 at (590.9, -229.9)
- removed the H37 at (662.1, -230.1)
- removed the H38 at (719.3, -230.2)
- removed the H39 at (762.4, -230.2)
- removed the H4 at (776.3, -354.1)
- removed the H40 at (828.7, -230.2)
- removed the H41 at (861.4, -230.2)
- removed the H42 at (899.5, -230.1)
- removed the H43 at (1003.7, -229.9)
- removed the H44 at (566.8, -209.3)
- removed the H45 at (610.0, -209.3)
- removed the H46 at (686.2, -209.5)
- removed the H47 at (757.3, -209.5)
- removed the H48 at (802.8, -209.5)
- removed the H49 at (861.4, -209.5)
- removed the H5 at (833.4, -354.1)
- removed the H50 at (918.4, -209.4)
- removed the H51 at (1003.7, -209.3)
- removed the H52 at (585.8, -333.2)
- removed the H53 at (623.9, -333.3)
- removed the H54 at (681.1, -333.4)
- removed the H55 at (738.2, -333.5)
- removed the H56 at (795.4, -333.5)
- removed the H57 at (832.4, -333.5)
- removed the H58 at (899.5, -333.4)
- removed the H6 at (918.7, -354.0)
- removed the H7 at (585.8, -312.6)
- removed the H8 at (642.9, -312.7)
- removed the H9 at (700.1, -312.8)
- removed the J1 at (771.5, -362.5)
- removed MX040: MX-NoLED, MX_Only:MXOnly-1.25U-Hotswap
- removed the NUM1 at (933.2, -340.6)
- removed the R4 at (934.4, -335.5)
- removed the R5 at (959.3, -335.5)
- removed the R6 at (984.4, -335.5)
- removed the SCRL1 at (983.1, -340.6)
- added MX100: 1U, HE60:MX-1U, F.Cu at (-51.0, -139.7)
- added MX77: 1U, HE60:MX-1U, F.Cu at (293.0, -79.7)
- added MX78: 1U, HE60:MX-1U, F.Cu at (273.9, -59.1)
- added MX79: 1U, HE60:MX-1U, F.Cu at (293.0, -59.1)
- added MX80: 1U, HE60:MX-1U, F.Cu at (312.0, -59.1)
- added MX81: 1U, HE60:MX-1U, F.Cu at (339.9, -141.4)
- added MX82: 1U, HE60:MX-1U, F.Cu at (359.0, -141.4)
- added MX83: 1U, HE60:MX-1U, F.Cu at (378.0, -141.4)
- added MX84: 1U, HE60:MX-1U, F.Cu at (397.1, -141.3)
- added MX85: 1U, HE60:MX-1U, F.Cu at (339.9, -120.8)
- added MX86: 1U, HE60:MX-1U, F.Cu at (359.0, -120.8)
- added MX87: 1U, HE60:MX-1U, F.Cu at (378.0, -120.8)
- added MX88: 1U, HE60:MX-1U, F.Cu at (397.1, -120.8)
- added MX89: 1U, HE60:MX-1U, F.Cu at (339.9, -100.2)
- added MX90: 1U, HE60:MX-1U, F.Cu at (359.0, -100.2)
- added MX91: 1U, HE60:MX-1U, F.Cu at (-51.0, -164.4)
- added MX92: 1U, HE60:MX-1U, F.Cu at (-51.0, -161.7)
- added MX93: 1U, HE60:MX-1U, F.Cu at (-51.0, -158.9)
- added MX94: 1U, HE60:MX-1U, F.Cu at (-51.0, -156.2)
- added MX95: 1U, HE60:MX-1U, F.Cu at (-51.0, -153.4)
- added MX96: 1U, HE60:MX-1U, F.Cu at (-51.0, -150.7)
- added MX97: 1U, HE60:MX-1U, F.Cu at (-51.0, -147.9)
- added MX98: 1U, HE60:MX-1U, F.Cu at (-51.0, -145.2)
- added MX99: 1U, HE60:MX-1U, F.Cu at (-51.0, -142.4)
- moved MX74 277.9 mm to (273.9, -120.8)
- moved MX75 276.9 mm to (292.9, -120.8)
- moved MX73 275.8 mm to (312.0, -141.4)
- moved MX76 275.6 mm to (312.0, -120.8)
- moved HE80 271.8 mm to (312.0, -59.1), turned to -90 degrees
- moved HE88 262.5 mm to (397.1, -120.8), turned to -90 degrees
- moved HE79 261.5 mm to (293.0, -59.1), turned to -90 degrees
- moved HE78 252.4 mm to (273.9, -59.1), turned to -90 degrees
- moved HE89 251.5 mm to (339.9, -100.2), turned to -90 degrees
- moved HE87 246.8 mm to (378.0, -120.8), turned to -90 degrees
- moved HE90 234.4 mm to (359.0, -100.2), turned to -90 degrees
- moved HE84 234.3 mm to (397.1, -141.3), turned to -90 degrees
- moved HE77 233.0 mm to (293.0, -79.7), turned to -90 degrees
- moved HE86 231.7 mm to (359.0, -120.8), turned to -90 degrees
- moved HE82 229.4 mm to (359.0, -141.4), turned to -90 degrees
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Routing:
- net HE88: vias 0 -> 1
- net GND: vias 53 -> 48
- removed copper zone on B.Cu, net +3.3V
Other:
- board size 1044 x 327.4 mm -> 447 x 162.8 mm

Commit message: feat: place everything*
Parts:
- removed C150, C151: 2.2u, Capacitor_SMD:C_0603_1608Metric
- removed C152, C153: 30p, Capacitor_SMD:C_0603_1608Metric
- removed C154, C155, C156, C158, C160, C225: 100n, Capacitor_SMD:C_0402_1005Metric
- removed C157: 10u, Capacitor_SMD:C_0603_1608Metric
- removed C159: 1u, Capacitor_SMD:C_0603_1608Metric
- removed C226: 4.7n, Capacitor_SMD:C_0402_1005Metric
- removed CAP1, NUM1, SCRL1: LED, LED_THT:LED_D3.0mm
- removed F1: BSMD0805-050-24V, Fuse:Fuse_0805_2012Metric
- removed HE101: MT9102ET, Package_TO_SOT_SMD:SOT-23-3
- removed the J1 at (-106.2, -460.2)
- removed the J1 at (174.5, -197.9)
- removed PCB1: H60, HE60:H60
- removed R4, R5, R6: 10K, Keebio-Parts:Resistor-Hybrid-Back
- removed R4: 12k, Resistor_SMD:R_0402_1005Metric
- removed SW1, SW2: TS-1187A-B-A-B, Button_Switch_SMD:SW_Push_1P1T_XKB_TS-1187A
- removed TH1, TH2: ToolingHole, HE60:ToolingHole
- removed U1: USBLC6-2SC6, Package_TO_SOT_SMD:SOT-23-6
- removed U2: TLV75733PDBV, Package_TO_SOT_SMD:SOT-23-5
- removed U3: XC6206P332MR-G, Package_TO_SOT_SMD:SOT-23-3
- removed U4: AT32F405RCT7, Package_QFP:LQFP-64_10x10mm_P0.5mm
- removed Y1: X322512MSB4SI, Crystal:Crystal_SMD_3225-4Pin_3.2x2.5mm
- added AM12: SN74LV4051A, Package_SO:TSSOP-16_4.4x5mm_P0.65mm, F.Cu at (306.6, -263.8)
- added AM13: SN74LV4051A, Package_SO:TSSOP-16_4.4x5mm_P0.65mm, F.Cu at (290.6, -265.3)
- added D1: LED, LED_THT:LED_D3.0mm, F.Cu at (336.2, -176.0)
- added D2: LED, LED_THT:LED_D3.0mm, F.Cu at (361.1, -176.0)
- added D3: LED, LED_THT:LED_D3.0mm, F.Cu at (386.2, -175.9)
- added J1: AudioJack3_Ground, Connector_Audio:Jack_3.5mm_PJ320E_Horizontal, F.Cu at (-19.1, -191.5)
- added RV1: R_Potentiometer_Trim_US, Potentiometer_THT:Potentiometer_Alpha_RD901F-40-00D_Single_Vertical, F.Cu at (11.6, -185.0)
- added RV10: R_Potentiometer_Trim_US, Potentiometer_THT:Potentiometer_Alpha_RD901F-40-00D_Single_Vertical, F.Cu at (202.1, -185.0)
- added RV11: R_Potentiometer_Trim_US, Potentiometer_THT:Potentiometer_Alpha_RD901F-40-00D_Single_Vertical, F.Cu at (221.2, -185.0)
- added RV12: R_Potentiometer_Trim_US, Potentiometer_THT:Potentiometer_Alpha_RD901F-40-00D_Single_Vertical, F.Cu at (240.2, -185.0)
- added RV2: R_Potentiometer_Trim_US, Potentiometer_THT:Potentiometer_Alpha_RD901F-40-00D_Single_Vertical, F.Cu at (30.6, -184.9)
- added RV3: R_Potentiometer_Trim_US, Potentiometer_THT:Potentiometer_Alpha_RD901F-40-00D_Single_Vertical, F.Cu at (49.7, -185.0)
- added RV4: R_Potentiometer_Trim_US, Potentiometer_THT:Potentiometer_Alpha_RD901F-40-00D_Single_Vertical, F.Cu at (68.8, -185.0)
- added RV5: R_Potentiometer_Trim_US, Potentiometer_THT:Potentiometer_Alpha_RD901F-40-00D_Single_Vertical, F.Cu at (97.4, -185.0)
- added RV6: R_Potentiometer_Trim_US, Potentiometer_THT:Potentiometer_Alpha_RD901F-40-00D_Single_Vertical, F.Cu at (116.4, -185.0)
- added RV7: R_Potentiometer_Trim_US, Potentiometer_THT:Potentiometer_Alpha_RD901F-40-00D_Single_Vertical, F.Cu at (135.5, -185.0)
- added RV8: R_Potentiometer_Trim_US, Potentiometer_THT:Potentiometer_Alpha_RD901F-40-00D_Single_Vertical, F.Cu at (154.5, -185.0)
- added RV9: R_Potentiometer_Trim_US, Potentiometer_THT:Potentiometer_Alpha_RD901F-40-00D_Single_Vertical, F.Cu at (183.1, -185.0)
- added SW3: RotaryEncoder_Switch, Rotary_Encoder:RotaryEncoder_Alps_EC11E_Vertical_H20mm, F.Cu at (266.4, -185.0)
- added SW4: RotaryEncoder_Switch, Rotary_Encoder:RotaryEncoder_Alps_EC11E_Vertical_H20mm, F.Cu at (285.5, -185.1)
- added SW5: RotaryEncoder_Switch, Rotary_Encoder:RotaryEncoder_Alps_EC11E_Vertical_H20mm, F.Cu at (304.6, -185.0)
- AM10, AM11, C161, C162, MX15: moved to F.Cu
- C148, C149: value 2.2u -> 100n; footprint Capacitor_SMD:C_0603_1608Metric -> Capacitor_SMD:C_0402_1005Metric
- J2: value JST_SH -> AudioJack3_Ground; footprint Connector_JST:JST_SH_SM04B-SRSS-TB_1x04-1MP_P1.00mm_Horizontal -> Connector_Audio:Jack_3.5mm_PJ320E_Horizontal
- MX55: value 15U -> 1U
- R1, R2: value 5.1k -> R_Small_US; footprint Resistor_SMD:R_0402_1005Metric -> Resistor_THT:R_Axial_DIN0204_L3.6mm_D1.6mm_P7.62mm_Horizontal
- R3: value 12k -> R_Small_US; footprint Resistor_SMD:R_0402_1005Metric -> Resistor_THT:R_Axial_DIN0204_L3.6mm_D1.6mm_P7.62mm_Horizontal; moved to F.Cu
- moved R2 567.8 mm to (358.6, -170.9)
- moved R1 547.6 mm to (333.6, -170.9)
- moved C148 491.9 mm to (312.4, -260.7)
- moved C149 491.6 mm to (312.4, -258.7)
- moved MX100 455.2 mm to (397.1, -59.1)
- moved MX96 453.7 mm to (397.1, -79.7)
- moved MX92 452.2 mm to (397.1, -100.2)
- moved MX99 437.0 mm to (378.0, -59.1)
- moved MX95 435.3 mm to (378.0, -79.7)
- moved MX91 433.8 mm to (378.0, -100.2)
- moved MX98 418.9 mm to (359.0, -59.1)
- moved MX94 417.0 mm to (359.0, -79.7)
- moved MX97 400.9 mm to (339.9, -59.1)
- moved MX93 398.8 mm to (339.9, -79.7)
- moved AM11 303.5 mm to (45.4, -239.8)
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Connections:
- A1 pad 10: unconnected-(A1-SPI1_POCI-Pad10) -> ENCODER_3_A
- A1 pad 11: unconnected-(A1-SPI1_PICO-Pad11) -> ENCODER_3_B
- A1 pad 16: unconnected-(A1-AUDIO_IN_1-Pad16) -> Audio_in_1
- A1 pad 17: unconnected-(A1-AUDIO_IN_2-Pad17) -> Audio_in_2
- A1 pad 18: unconnected-(A1-AUDIO_OUT_1-Pad18) -> Audio_out_1
- A1 pad 19: unconnected-(A1-AUDIO_OUT_2-Pad19) -> Audio_out_2
- A1 pad 3: unconnected-(A1-SD_DATA_2-Pad3) -> ENB_B
- A1 pad 32: MUX_OUT_11 -> MUX_OUT_12
- A1 pad 33: unconnected-(A1-SAI2_SD_A-Pad33) -> ENCODER_1_Btn
- A1 pad 34: unconnected-(A1-SAI2_FS-Pad34) -> ENCODER_2_Btn
- A1 pad 36: unconnected-(A1-USB_D_--Pad36) -> ENCODER_3_Btn
- A1 pad 4: unconnected-(A1-SD_DATA_1-Pad4) -> ENB_A
- A1 pad 6: unconnected-(A1-SD_CMD-Pad6) -> ENCODER_1_A
- A1 pad 7: unconnected-(A1-SD_CLK-Pad7) -> ENCODER_1_B
- A1 pad 8: unconnected-(A1-SPI1_CS-Pad8) -> ENCODER_2_A
- A1 pad 9: unconnected-(A1-SPI1_SCK-Pad9) -> ENCODER_2_B
- AM1 pad 1: HE5 -> HE1
- AM1 pad 12: GND -> HE8
- AM1 pad 13: HE4 -> HE7
- AM1 pad 14: HE3 -> HE6
- AM1 pad 15: HE2 -> HE5
- AM1 pad 2: HE6 -> HE2
- AM1 pad 4: HE7 -> HE3
- AM1 pad 5: HE8 -> HE4
- AM11 pad 1: unconnected-(AM11-X4-Pad1) -> HE1
- AM11 pad 12: unconnected-(AM11-X3-Pad12) -> HE8
- AM11 pad 13: unconnected-(AM11-X0-Pad13) -> HE7
- AM11 pad 14: unconnected-(AM11-X1-Pad14) -> HE6
- AM11 pad 15: unconnected-(AM11-X2-Pad15) -> HE5
- AM11 pad 2: unconnected-(AM11-X6-Pad2) -> HE2
- AM11 pad 3: MUX_OUT_11 -> MUX_OUT_10
- AM11 pad 4: unconnected-(AM11-X7-Pad4) -> HE3
- AM11 pad 5: unconnected-(AM11-X5-Pad5) -> HE4
- AM3 pad 1: HE20 -> HE17
- AM3 pad 12: HE19 -> HE24
- AM3 pad 13: HE18 -> HE23
- AM3 pad 14: HE17 -> HE22
- AM3 pad 15: HE1 -> HE21
- AM3 pad 2: GND -> HE18
- AM3 pad 4: HE21 -> HE19
- AM3 pad 5: HE22 -> HE20
- AM4 pad 1: HE23 -> HE25
- AM4 pad 12: HE30 -> HE32
- AM4 pad 13: HE29 -> HE31
- AM4 pad 14: HE28 -> HE30
- AM4 pad 15: HE27 -> HE29
- AM4 pad 2: HE24 -> HE26
- AM4 pad 4: HE25 -> HE27
- AM4 pad 5: HE26 -> HE28
- AM5 pad 1: HE32 -> HE33
- AM5 pad 12: HE38 -> HE40
- AM5 pad 13: HE37 -> HE39
- AM5 pad 14: HE36 -> HE38
- AM5 pad 15: GND -> HE37
- AM5 pad 2: HE33 -> HE34
- AM5 pad 4: HE34 -> HE35
- AM5 pad 5: HE35 -> HE36
- AM6 pad 1: HE39 -> HE41
- AM6 pad 12: HE55 -> HE48
- AM6 pad 13: HE56 -> HE47
- AM6 pad 14: HE57 -> HE46
- AM6 pad 15: HE43 -> HE45
- AM6 pad 2: HE40 -> HE42
- AM6 pad 4: HE41 -> HE43
- AM6 pad 5: HE42 -> HE44
- AM7 pad 1: HE31 -> HE49
- AM7 pad 12: HE61 -> unconnected-(AM7-X3-Pad12)
- AM7 pad 13: HE60 -> unconnected-(AM7-X0-Pad13)
- AM7 pad 14: HE59 -> unconnected-(AM7-X1-Pad14)
- AM7 pad 15: HE58 -> unconnected-(AM7-X2-Pad15)
- AM7 pad 2: HE44 -> unconnected-(AM7-X6-Pad2)
- AM7 pad 4: HE45 -> unconnected-(AM7-X7-Pad4)
- AM7 pad 5: HE46 -> unconnected-(AM7-X5-Pad5)
- AM8 pad 1: HE47 -> unconnected-(AM8-X4-Pad1)
- AM8 pad 12: HE62 -> unconnected-(AM8-X3-Pad12)
- AM8 pad 13: HE63 -> unconnected-(AM8-X0-Pad13)
- AM8 pad 14: HE64 -> unconnected-(AM8-X1-Pad14)
- AM8 pad 15: HE65 -> unconnected-(AM8-X2-Pad15)
- AM8 pad 2: HE48 -> unconnected-(AM8-X6-Pad2)
- AM8 pad 4: HE49 -> unconnected-(AM8-X7-Pad4)
- AM8 pad 5: HE50 -> unconnected-(AM8-X5-Pad5)
- C148 pad 1: +5V -> +3.3VA
- R1 pad 2: GND -> unconnected-(R1-Pad2)
- R2 pad 1: GND -> Net-(D2-A)
- R2 pad 2: Net-(J1-CC2) -> unconnected-(R2-Pad2)
- R3 pad 1: GND -> Net-(D3-A)
- R3 pad 2: Net-(U4-OTGHS1_R) -> unconnected-(R3-Pad2)
Routing:
- net +3.3VA: track 0.00 -> 2297.9 mm, vias 3 -> 0
- net HE8: track 0.00 -> 78.3 mm
- net HE1: track 0.00 -> 71.4 mm
- net HE14: track 0.00 -> 63.6 mm
- net HE7: track 0.00 -> 60.9 mm
- net HE9: track 0.00 -> 50.8 mm
- net HE2: track 0.00 -> 48.9 mm
- net HE6: track 0.00 -> 42.4 mm
- net HE13: track 0.00 -> 40.5 mm
- net HE10: track 0.00 -> 32.7 mm
- net HE3: track 0.00 -> 32.3 mm
- net HE5: track 0.00 -> 23.3 mm
- net HE12: track 0.00 -> 17.0 mm
- net HE11: track 0.00 -> 15.5 mm
- net HE4: track 0.00 -> 14.3 mm
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