File: keyboard_keyboard/kicad/keyboard_keyboard.kicad_pcb (KiCad board)
At the start: 2 copper layers, 447 x 162.8 mm, 504 parts, among them J1 AudioJack3_Ground, J2 AudioJack3_Ground, SW3 RotaryEncoder_Switch, SW4 RotaryEncoder_Switch, SW5 RotaryEncoder_Switch

Commit message: update wires
Parts:
- removed SW3, SW4, SW5: RotaryEncoder_Switch, Rotary_Encoder:RotaryEncoder_Alps_EC11E_Vertical_H20mm
- added AM14: SN74LV4051A, Package_SO:TSSOP-16_4.4x5mm_P0.65mm, B.Cu at (84.0, -157.4)
- added AM15: SN74LV4051A, Package_SO:TSSOP-16_4.4x5mm_P0.65mm, B.Cu at (215.9, -163.9)
- added C150: 100n, Capacitor_SMD:C_0402_1005Metric, B.Cu at (280.1, -271.7)
- added C151: 100n, Capacitor_SMD:C_0402_1005Metric, B.Cu at (282.1, -271.7)
- added J3: Screen Connector, Connector_PinHeader_2.54mm:PinHeader_1x04_P2.54mm_Vertical, F.Cu at (268.5, -185.8)
- AM10, AM11, AM12, AM13, C148, C149: moved to B.Cu
- moved AM10 296.8 mm to (324.5, -134.5), turned to -90 degrees
- moved AM11 284.9 mm to (292.7, -98.4), turned to -90 degrees
- moved C145 222.5 mm to (288.0, -241.9)
- moved C146 222.5 mm to (288.0, -239.9)
- moved C161 222.5 mm to (288.0, -238.0)
- moved C162 222.5 mm to (288.0, -236.0)
- moved AM13 209.5 mm to (368.7, -70.9), turned to -90 degrees
- moved AM12 164.9 mm to (368.2, -110.9), turned to -90 degrees
- moved AM9 81.4 mm to (74.5, -49.0)
- moved AM8 74.0 mm to (189.0, -68.5)
- moved C148 58.9 mm to (270.8, -218.9), turned to -90 degrees
- moved C149 56.1 mm to (272.8, -218.9), turned to -90 degrees
- moved A1 52.7 mm to (417.5, -239.6)
- moved AM4 33.1 mm to (179.0, -111.5)
- moved AM5 21.5 mm to (55.7, -90.9)
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Connections:
- A1 pad 10: ENCODER_3_A -> MUX_SELECT_2
- A1 pad 11: ENCODER_3_B -> unconnected-(A1-SPI1_PICO-Pad11)
- A1 pad 12: unconnected-(A1-I2C1_SCL-Pad12) -> SCL
- A1 pad 13: unconnected-(A1-I2C1_SDA-Pad13) -> SDA
- A1 pad 2: unconnected-(A1-SD_DATA_3-Pad2) -> ENB_C
- A1 pad 20: unconnected-(A1-AGND-Pad20) -> GND
- A1 pad 33: ENCODER_1_Btn -> MUX_OUT_14
- A1 pad 34: ENCODER_2_Btn -> unconnected-(A1-SAI2_FS-Pad34)
- A1 pad 36: ENCODER_3_Btn -> unconnected-(A1-USB_D_--Pad36)
- A1 pad 38: unconnected-(A1-3V3_D-Pad38) -> +3.3VA
- A1 pad 40: unconnected-(A1-DGND-Pad40) -> GND
- A1 pad 6: ENCODER_1_A -> unconnected-(A1-SD_CMD-Pad6)
- A1 pad 7: ENCODER_1_B -> unconnected-(A1-SD_CLK-Pad7)
- A1 pad 8: ENCODER_2_A -> MUX_SELECT_0
- A1 pad 9: ENCODER_2_B -> MUX_SELECT_1
- AM10 pad 1: HE74 -> HE71
- AM10 pad 12: HE70 -> GND
- AM10 pad 13: HE73 -> HE84
- AM10 pad 14: HE72 -> HE83
- AM10 pad 15: HE71 -> HE82
- AM10 pad 2: HE75 -> HE72
- AM10 pad 4: HE76 -> HE73
- AM10 pad 5: HE77 -> HE81
- AM10 pad 6: GND -> ENABLE_10
- AM11 pad 1: HE1 -> HE74
- AM11 pad 12: HE8 -> GND
- AM11 pad 13: HE7 -> HE80
- AM11 pad 14: HE6 -> HE79
- AM11 pad 15: HE5 -> HE78
- AM11 pad 2: HE2 -> HE75
- AM11 pad 4: HE3 -> HE76
- AM11 pad 5: HE4 -> HE77
- AM11 pad 6: GND -> ENABLE_11
- AM12 pad 1: unconnected-(AM12-X4-Pad1) -> HE85
- AM12 pad 12: unconnected-(AM12-X3-Pad12) -> HE92
- AM12 pad 13: unconnected-(AM12-X0-Pad13) -> HE91
- AM12 pad 14: unconnected-(AM12-X1-Pad14) -> HE90
- AM12 pad 15: unconnected-(AM12-X2-Pad15) -> HE89
- AM12 pad 2: unconnected-(AM12-X6-Pad2) -> HE86
- AM12 pad 4: unconnected-(AM12-X7-Pad4) -> HE87
- AM12 pad 5: unconnected-(AM12-X5-Pad5) -> HE88
- AM12 pad 6: GND -> ENABLE_12
- AM13 pad 1: unconnected-(AM13-X4-Pad1) -> HE93
- AM13 pad 12: unconnected-(AM13-X3-Pad12) -> HE100
- AM13 pad 13: unconnected-(AM13-X0-Pad13) -> HE99
- AM13 pad 14: unconnected-(AM13-X1-Pad14) -> HE98
- AM13 pad 15: unconnected-(AM13-X2-Pad15) -> HE97
- AM13 pad 2: unconnected-(AM13-X6-Pad2) -> HE94
- AM13 pad 4: unconnected-(AM13-X7-Pad4) -> HE95
- AM13 pad 5: unconnected-(AM13-X5-Pad5) -> HE96
- AM13 pad 6: GND -> ENABLE_13
- AM2 pad 12: HE16 -> HE28
- AM2 pad 13: HE15 -> HE29
- AM3 pad 1: HE17 -> HE15
- AM3 pad 12: HE24 -> HE22
- AM3 pad 13: HE23 -> HE21
- AM3 pad 14: HE22 -> HE20
- AM3 pad 15: HE21 -> HE19
- AM3 pad 2: HE18 -> HE16
- AM3 pad 4: HE19 -> HE17
- AM3 pad 5: HE20 -> HE18
- AM4 pad 1: HE25 -> HE23
- AM4 pad 12: HE32 -> HE43
- AM4 pad 13: HE31 -> HE42
- AM4 pad 14: HE30 -> HE41
- AM4 pad 15: HE29 -> HE27
- AM4 pad 2: HE26 -> HE24
- AM4 pad 4: HE27 -> HE25
- AM4 pad 5: HE28 -> HE26
- AM5 pad 1: HE33 -> HE30
- AM5 pad 12: HE40 -> HE37
- AM5 pad 13: HE39 -> HE36
- AM5 pad 14: HE38 -> HE35
- AM5 pad 15: HE37 -> HE34
- AM5 pad 2: HE34 -> HE31
- AM5 pad 4: HE35 -> HE32
- AM5 pad 5: HE36 -> HE33
- AM6 pad 1: HE41 -> HE38
- AM6 pad 12: HE48 -> HE58
- AM6 pad 13: HE47 -> HE57
- AM6 pad 14: HE46 -> HE56
- AM6 pad 15: HE45 -> HE55
- AM6 pad 2: HE42 -> HE39
- AM6 pad 4: HE43 -> HE40
- AM6 pad 5: HE44 -> HE54
- AM7 pad 1: HE49 -> HE44
- AM7 pad 12: unconnected-(AM7-X3-Pad12) -> HE51
- AM7 pad 13: unconnected-(AM7-X0-Pad13) -> HE50
- AM7 pad 14: unconnected-(AM7-X1-Pad14) -> HE49
- AM7 pad 15: unconnected-(AM7-X2-Pad15) -> HE48
- AM7 pad 2: unconnected-(AM7-X6-Pad2) -> HE45
- AM7 pad 4: unconnected-(AM7-X7-Pad4) -> HE46
- AM7 pad 5: unconnected-(AM7-X5-Pad5) -> HE47
- AM8 pad 1: unconnected-(AM8-X4-Pad1) -> HE52
- AM8 pad 12: unconnected-(AM8-X3-Pad12) -> GND
- AM8 pad 13: unconnected-(AM8-X0-Pad13) -> GND
- AM8 pad 14: unconnected-(AM8-X1-Pad14) -> HE70
- AM8 pad 15: unconnected-(AM8-X2-Pad15) -> HE69
- AM8 pad 2: unconnected-(AM8-X6-Pad2) -> HE53
- AM8 pad 4: unconnected-(AM8-X7-Pad4) -> HE67
- AM8 pad 5: unconnected-(AM8-X5-Pad5) -> HE68
- AM9 pad 1: HE51 -> HE59
- AM9 pad 13: HE67 -> HE65
- AM9 pad 14: HE68 -> HE64
- AM9 pad 15: HE69 -> HE63
- AM9 pad 2: HE52 -> HE60
- AM9 pad 4: HE53 -> HE61
- AM9 pad 5: HE54 -> HE62
- C198 pad 1: HE86 -> HE87
- HE87 pad 2: HE86 -> HE87
Routing:
- net MUX_SELECT_0: track 0.00 -> 493.7 mm, vias 0 -> 16
- net MUX_SELECT_2: track 0.00 -> 491.9 mm, vias 0 -> 16
- net MUX_SELECT_1: track 0.00 -> 491.1 mm, vias 0 -> 16
- net +3.3VA: track 2297.9 -> 2685.5 mm, vias 0 -> 2
- net HE59: track 3.25 -> 93.2 mm
- net POT1: track 0.00 -> 89.1 mm
- net POT8: track 0.00 -> 82.8 mm
- net HE84: track 1.99 -> 84.3 mm
- net HE44: track 1.99 -> 80.1 mm
- net HE66: track 2.30 -> 79.3 mm
- net HE37: track 1.99 -> 77.9 mm
- net HE15: track 2.16 -> 77.9 mm
- net POT2: track 0.00 -> 73.1 mm
- net HE30: track 1.99 -> 74.5 mm
- net HE58: track 2.50 -> 74.1 mm
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
Commit message: routes
Parts:
- added U1: 74HC138, Package_SO:SOIC-16_3.9x9.9mm_P1.27mm, B.Cu at (349.5, -161.1)
- A1, C145, C146, C161, C162: moved to B.Cu
- moved J1 418.7 mm to (399.3, -177.6), turned to -90 degrees
- moved J2 403.7 mm to (399.8, -165.5), turned to -90 degrees
- moved C145 296.6 mm to (50.0, -65.0), turned to -90 degrees
- moved C150 233.2 mm to (79.0, -153.5)
- moved C146 203.7 mm to (184.5, -64.5), turned to -90 degrees
- moved C149 177.0 mm to (364.5, -67.5)
- moved C148 145.3 mm to (364.0, -107.5)
- moved C162 142.0 mm to (288.0, -94.0), turned to -90 degrees
- moved C151 132.8 mm to (211.0, -159.5)
- moved C161 109.4 mm to (320.5, -133.5), turned to -90 degrees
- moved C147 84.1 mm to (70.0, -46.0)
- moved C144 79.8 mm to (174.5, -86.0)
- moved A1 57.9 mm to (408.2, -182.5), turned to 90 degrees
- moved C139 49.0 mm to (50.5, -126.5)
- moved C143 46.8 mm to (51.0, -88.0)
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Connections:
- A1 pad 2: ENB_C -> led_3
- A1 pad 3: ENB_B -> ENB_C
- A1 pad 4: ENB_A -> ENB_B
- A1 pad 5: unconnected-(A1-SD_DATA_0-Pad5) -> ENB_A
- A1 pad 6: unconnected-(A1-SD_CMD-Pad6) -> led_2
- A1 pad 7: unconnected-(A1-SD_CLK-Pad7) -> led_1
- D1 pad 1: unconnected-(D1-K-Pad1) -> led_1
- D2 pad 1: unconnected-(D2-K-Pad1) -> led_2
- D3 pad 1: unconnected-(D3-K-Pad1) -> led_3
- R1 pad 2: unconnected-(R1-Pad2) -> +3.3VA
- R2 pad 2: unconnected-(R2-Pad2) -> +3.3VA
- R3 pad 2: unconnected-(R3-Pad2) -> +3.3VA
Routing:
- net MUX_SELECT_1: track 491.1 -> 923.0 mm
- net MUX_SELECT_0: track 493.7 -> 922.8 mm
- net +3.3VA: track 2685.5 -> 3060.8 mm
- net ENABLE_14: track 0.00 -> 278.4 mm, vias 0 -> 2
- net MUX_SELECT_2: track 491.9 -> 723.5 mm
- net ENABLE_15: track 0.00 -> 141.6 mm, vias 0 -> 2
- net ENABLE_13: track 0.00 -> 137.5 mm, vias 0 -> 2
- net ENABLE_12: track 0.00 -> 98.9 mm, vias 0 -> 2
- net ENABLE_11: track 0.00 -> 90.7 mm, vias 0 -> 2
- net led_1: track 0.00 -> 60.6 mm
- net led_2: track 0.00 -> 37.1 mm
- net ENABLE_10: track 0.00 -> 30.3 mm, vias 0 -> 2
- net led_3: track 0.00 -> 22.2 mm
- net Net-(D3-A): track 0.00 -> 7.18 mm
- net Net-(D1-A): track 0.00 -> 7.17 mm
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
Commit message: more routes
Routing:
- net MUX_OUT_9: track 0.00 -> 461.9 mm, vias 0 -> 1
- net MUX_OUT_7: track 0.00 -> 416.2 mm, vias 0 -> 1
- net MUX_OUT_5: track 0.00 -> 389.6 mm, vias 0 -> 1
- net MUX_OUT_3: track 0.00 -> 364.9 mm, vias 0 -> 1
- net +3.3VA: track 3060.8 -> 3157.7 mm
- net POT5: track 39.4 -> 51.4 mm
- net ENABLE_14: track 278.4 -> 273.9 mm
- net MUX_SELECT_1: track 923.0 -> 925.3 mm
- net POT8: track 82.8 -> 85.2 mm
- net ENABLE_12: track 98.9 -> 96.8 mm
- net POT6: track 49.9 -> 51.7 mm
- net HE47: track 23.5 -> 24.7 mm
- net MUX_SELECT_0: track 922.8 -> 924.0 mm
- net MUX_SELECT_2: track 723.5 -> 724.6 mm
- net HE46: track 43.0 -> 44.0 mm
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
Commit message: wire more stuff
Routing:
- net MUX_OUT_1: track 0.00 -> 343.6 mm, vias 0 -> 1
- net MUX_OUT_14: track 0.00 -> 343.4 mm, vias 0 -> 2
- net MUX_OUT_8: track 0.00 -> 306.7 mm, vias 0 -> 3
- net MUX_OUT_12: track 0.00 -> 223.5 mm, vias 0 -> 2
- net MUX_OUT_10: track 0.00 -> 156.5 mm, vias 0 -> 3
- net MUX_OUT_6: track 0.00 -> 147.3 mm, vias 0 -> 2
- net MUX_OUT_4: track 0.00 -> 112.3 mm, vias 0 -> 2
- net MUX_OUT_2: track 0.00 -> 89.3 mm, vias 0 -> 2
- net MUX_SELECT_2: track 724.6 -> 805.6 mm, vias 16 -> 18
- net +3.3VA: track 3157.7 -> 3236.2 mm
- net ENB_C: track 0.00 -> 64.9 mm, vias 0 -> 1
- net ENB_B: track 0.00 -> 63.5 mm, vias 0 -> 1
- net ENB_A: track 0.00 -> 62.6 mm, vias 0 -> 1
- net ENABLE_12: track 96.8 -> 103.9 mm
- net ENABLE_13: track 137.5 -> 144.0 mm
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