File: keyboard_keyboard/kicad/keyboard_keyboard.kicad_pcb (KiCad board)
At the start: 2 copper layers, 447 x 162.8 mm, 507 parts, among them J1 AudioJack3_Ground, J2 AudioJack3_Ground, J3 Screen Connector, U1 74HC138

Commit message: more routes
Connections:
- J1 pad R1: (no net) -> Audio_in_2
- J1 pad R2: (no net) -> GND
- J2 pad R1: (no net) -> Audio_out_2
- J2 pad R2: (no net) -> GND
Routing:
- net MUX_OUT_2: track 89.3 -> 222.8 mm, vias 2 -> 3
- net MUX_OUT_6: track 147.3 -> 280.9 mm, vias 2 -> 3
- net MUX_OUT_4: track 112.3 -> 245.2 mm, vias 2 -> 3
- net SCL: track 0.00 -> 113.5 mm
- net SDA: track 0.00 -> 110.4 mm
- net Audio_out_2: track 0.00 -> 75.9 mm
- net Audio_out_1: track 0.00 -> 73.8 mm
- net MUX_SELECT_0: track 925.9 -> 988.1 mm, vias 16 -> 18
- net MUX_SELECT_1: track 927.5 -> 987.4 mm, vias 16 -> 18
- net Audio_in_2: track 0.00 -> 59.3 mm
- net Audio_in_1: track 0.00 -> 58.8 mm
- net MUX_OUT_8: track 306.7 -> 309.9 mm
- net +3.3VA: track 3236.2 -> 3233.2 mm
- net MUX_OUT_1: track 343.6 -> 341.2 mm
- net MUX_OUT_3: track 368.7 -> 366.9 mm
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